File: PCB/Build Pad.kicad_pcb (KiCad board)
At the start: 2 copper layers, 95 x 73.5 mm, 30 parts, among them SW1 SW_Push, SW2 SW_Push, SW3 SW_Push, SW4 SW_Push, SW5 SW_Push, SW6 SW_Push, SW7 RotaryEncoder_Switch, U1 XIAO-RP2040-DIP

Commit message: Add files via upload
Parts:
- moved U1 5.12 mm to (184.8, 59.1)
- moved OLED1 1.54 mm to (113.7, 56.5)
Routing:
- net /D7: track 44.6 -> 37.5 mm
- net /ROW2: track 160.3 -> 153.3 mm
- net /D6: track 87.6 -> 80.6 mm
- net /ROW1: track 108.4 -> 114.6 mm
- net /RGB: track 114.7 -> 120.7 mm
- net /D9: track 77.3 -> 82.5 mm
- net +3.3V: track 92.6 -> 97.8 mm
- net /COL3: track 116.1 -> 111.1 mm
- net +5V: track 251.1 -> 254.1 mm
- net /COL1: track 166.4 -> 163.5 mm
- net /COL2: track 137.5 -> 135.3 mm
- net /D5: track 38.6 -> 37.9 mm
